File: Matrix.sch (KiCad schematic (older format))
At the start: 90 parts

Commit message: Final touches on schematic & Clean up PCB
Parts:
- D1, D10, D11, D12, D13, D14, D15, D16, D17, D18, D19, D2, D20, D21, D22, D23, D24, D25, D26, D27, D28, D29, D3, D30, D31, D32, D321, D33, D331, D34, D35, D36, D37, D38, D381, D39, D4, D40, D41, D42, D5, D6, D7, D8, D9: footprint SM0805:SM0805D -> Diodes_SMD:SOD-123
- S1, S10, S11, S12, S13, S14, S15, S16, S17, S18, S19, S2, S20, S21, S22, S23, S24, S25, S26, S27, S28, S29, S3, S30, S31, S32, S321, S33, S331, S34, S35, S36, S37, S38, S381, S39, S4, S40, S41, S42, S5, S6, S7, S8, S9: footprint MX1A_alps:MX1ALPS -> mx1a:MX1A
Connections:
- wire segments 243 -> 153

Commit message: Layout
Parts:
- removed D321, D331, D381: DIODE, Diodes_SMD:SOD-123, symbol DIODE
- added S361, S401: MX1A, mx1a:MX1A, symbol MX1A
Connections:
- wire segments 153 -> 156
Other:
- moved on the sheet: D32, D33, D36, D38, D40, S321, S331, S381
Changed lines of the file:
@@
-$EndComp
-$Comp
-L DIODE D32
-U 1 1 5740CB82
-P 8250 4350
-F 0 "D32" H 8250 4250 40  0000 C CNN
-F 1 "DIODE" H 8250 4250 40  0001 C CNN
-F 2 "Diodes_SMD:SOD-123" H 8250 4350 60  0001 C CNN
-F 3 "" H 8250 4350 60  0000 C CNN
-	1    8250 4350
-	1    0    0    -1
 $EndComp
 $Comp
@@
 L DIODE D33
 U 1 1 5740CB91
-P 8850 4350
-F 0 "D33" H 8850 4250 40  0000 C CNN
-F 1 "DIODE" H 8850 4250 40  0001 C CNN
-F 2 "Diodes_SMD:SOD-123" H 8850 4350 60  0001 C CNN
-F 3 "" H 8850 4350 60  0000 C CNN
-	1    8850 4350
+P 8750 4600
+F 0 "D33" H 8750 4500 40  0000 C CNN
+F 1 "DIODE" H 8750 4500 40  0001 C CNN
+F 2 "Diodes_SMD:SOD-123" H 8750 4600 60  0001 C CNN
+F 3 "" H 8750 4600 60  0000 C CNN
+	1    8750 4600
 	1    0    0    -1
 $EndComp
@@
 L DIODE D36
 U 1 1 5740CBBE
-P 3850 5550
-F 0 "D36" H 3850 5450 40  0000 C CNN
-F 1 "DIODE" H 3850 5450 40  0001 C CNN
-F 2 "Diodes_SMD:SOD-123" H 3850 5550 60  0001 C CNN
-F 3 "" H 3850 5550 60  0000 C CNN
-	1    3850 5550
+P 3750 5850
+F 0 "D36" H 3750 5750 40  0000 C CNN
+F 1 "DIODE" H 3750 5750 40  0001 C CNN
+F 2 "Diodes_SMD:SOD-123" H 3750 5850 60  0001 C CNN
+F 3 "" H 3750 5850 60  0000 C CNN
+	1    3750 5850
 	1    0    0    -1
 $EndComp
@@
 L DIODE D38
 U 1 1 5740CBEB
-P 5750 5550
-F 0 "D38" H 5750 5450 40  0000 C CNN
-F 1 "DIODE" H 5750 5450 40  0001 C CNN
-F 2 "Diodes_SMD:SOD-123" H 5750 5550 60  0001 C CNN
-F 3 "" H 5750 5550 60  0000 C CNN
-	1    5750 5550
+P 5650 5850
+F 0 "D38" H 5650 5750 40  0000 C CNN
+F 1 "DIODE" H 5650 5750 40  0001 C CNN
+F 2 "Diodes_SMD:SOD-123" H 5650 5850 60  0001 C CNN
+F 3 "" H 5650 5850 60  0000 C CNN
+	1    5650 5850
 	1    0    0    -1
 $EndComp
@@
 L DIODE D40
 U 1 1 5740CC18
-P 7600 5550
-F 0 "D40" H 7600 5450 40  0000 C CNN
-F 1 "DIODE" H 7600 5450 40  0001 C CNN
-F 2 "Diodes_SMD:SOD-123" H 7600 5550 60  0001 C CNN
-F 3 "" H 7600 5550 60  0000 C CNN
-	1    7600 5550
+P 7500 5850
+F 0 "D40" H 7500 5750 40  0000 C CNN
+F 1 "DIODE" H 7500 5750 40  0001 C CNN
+F 2 "Diodes_SMD:SOD-123" H 7500 5850 60  0001 C CNN
+F 3 "" H 7500 5850 60  0000 C CNN
+	1    7500 5850
 	1    0    0    -1
 $EndComp
@@
 L MX1A S381
 U 1 1 586CA3F7
-P 5650 6000
-F 0 "S381" H 5500 6250 60  0000 C CNN
-F 1 "MX1A" H 5650 6100 60  0000 C CNN
-F 2 "mx1a:MX1A" H 5650 6000 60  0001 C CNN
-F 3 "" H 5650 6000 60  0000 C CNN
-	1    5650 6000
-	1    0    0    -1
-$EndComp
-$Comp
-L DIODE D381
-U 1 1 586CA3FE
-P 5650 6000
-F 0 "D381" H 5650 5900 40  0000 C CNN
-F 1 "DIODE" H 5650 5900 40  0001 C CNN
-F 2 "Diodes_SMD:SOD-123" H 5650 6000 60  0001 C CNN
-F 3 "" H 5650 6000 60  0000 C CNN
-	1    5650 6000
+P 5650 5800
+F 0 "S381" H 5500 6050 60  0000 C CNN
+F 1 "MX1A" H 5650 5900 60  0000 C CNN
+F 2 "mx1a:MX1A" H 5650 5800 60  0001 C CNN
+F 3 "" H 5650 5800 60  0000 C CNN
+	1    5650 5800
 	1    0    0    -1
 $EndComp
@@
 	1    0    0    -1
 $EndComp
-$Comp
-L MX1A S321
-U 1 1 586CD089
-P 8150 4800
-F 0 "S321" H 8000 5050 60  0000 C CNN
-F 1 "MX1A" H 8150 4900 60  0000 C CNN
-F 2 "mx1a:MX1A" H 8150 4800 60  0001 C CNN
-F 3 "" H 8150 4800 60  0000 C CNN
-	1    8150 4800
-	1    0    0    -1
-$EndComp
-$Comp
-L DIODE D321
-U 1 1 586CD090
-P 8150 4800
-F 0 "D321" H 8150 4700 40  0000 C CNN
-F 1 "DIODE" H 8150 4700 40  0001 C CNN
-F 2 "Diodes_SMD:SOD-123" H 8150 4800 60  0001 C CNN
-F 3 "" H 8150 4800 60  0000 C CNN
-	1    8150 4800
-	1    0    0    -1
-$EndComp
-$Comp
-L MX1A S331
-U 1 1 586CDBF9
-P 8750 4800
-F 0 "S331" H 8600 5050 60  0000 C CNN
-F 1 "MX1A" H 8750 4900 60  0000 C CNN
-F 2 "mx1a:MX1A" H 8750 4800 60  0001 C CNN
-F 3 "" H 8750 4800 60  0000 C CNN
-	1    8750 4800
-	1    0    0    -1
-$EndComp
-$Comp
-L DIODE D331
-U 1 1 586CDC00
-P 8750 4800
-F 0 "D331" H 8750 4700 40  0000 C CNN
-F 1 "DIODE" H 8750 4700 40  0001 C CNN
-F 2 "Diodes_SMD:SOD-123" H 8750 4800 60  0001 C CNN
-F 3 "" H 8750 4800 60  0000 C CNN
-	1    8750 4800
-	1    0    0    -1
-$EndComp
 Wire Wire Line
 	2800 2050 2800 2200
@@
 	7400 4500 7900 4500
 Wire Wire Line
-	8450 4200 8450 4350
-Wire Wire Line
-	8050 4350 8050 4500
-Wire Wire Line
-	8050 4500 8500 4500
-Wire Wire Line
-	9050 4200 9050 4350
-Wire Wire Line
-	8650 4350 8650 4500
-Wire Wire Line
-	8650 4500 9100 4500
+	8450 4200 8450 4600
+Wire Wire Line
+	9050 4200 9050 4600
 Wire Wire Line
 	2800 5400 2800 5550
@@
 	3050 5700 3500 5700
 Wire Wire Line
-	4050 5400 4050 5550
-Wire Wire Line
-	3650 5550 3650 5700
-Wire Wire Line
-	3650 5700 4150 5700
-Wire Wire Line
-	5950 5400 5950 5550
-Wire Wire Line
-	5550 5550 5550 5700
-Wire Wire Line
-	5550 5700 6000 5700
-Wire Wire Line
-	7800 5400 7800 5550
-Wire Wire Line
-	7400 5550 7400 5700
-Wire Wire Line
-	7400 5700 7900 5700
+	4050 5400 4050 5850
+Wire Wire Line
+	3550 5850 3550 6000
+Wire Wire Line
+	3550 6000 4150 6000
+Wire Wire Line
+	5950 5400 5950 5850
+Wire Wire Line
+	7800 5400 7800 5850
+Wire Wire Line
+	7300 5850 7300 6000
+Wire Wire Line
+	7300 6000 7900 6000
 Wire Wire Line
 	8450 5400 8450 5550
@@
 	9100 1350 9100 6300
 Connection ~ 9100 5700
-Connection ~ 9100 4500
 Connection ~ 9100 3350
 Connection ~ 9100 2350
@@
 Connection ~ 3500 4500
 Connection ~ 4150 4500
-Connection ~ 4150 5700
+Connection ~ 4150 6000
 Connection ~ 4150 3350
 Connection ~ 4150 2350
@@
 Connection ~ 6000 3350
 Connection ~ 6000 4500
-Connection ~ 6000 5700
 Connection ~ 6650 2350
 Connection ~ 6650 3350
@@
 Connection ~ 7900 3350
 Connection ~ 7900 4500
-Connection ~ 7900 5700
+Connection ~ 7900 6000
 Connection ~ 8500 5700
-Connection ~ 8500 4500
 Connection ~ 8500 3350
 Connection ~ 2400 1800
@@
 	8650 5550 8650 5700
 Wire Wire Line
-	5850 5850 5850 6000
-Wire Wire Line
-	5450 6000 5450 6150
-Wire Wire Line
-	5450 6150 6000 6150
-Wire Wire Line
-	5450 5600 5450 5150
+	5450 5400 5450 5150
 Connection ~ 5450 5150
-Connection ~ 6000 6150
 Wire Wire Line
 	4950 5550 4950 5700
@@
 Connection ~ 5400 5700
 Wire Wire Line
-	8350 4650 8350 4800
-Wire Wire Line
-	7950 4800 7950 4950
-Wire Wire Line
-	7950 4950 8500 4950
-Connection ~ 8500 4950
-Wire Wire Line
-	7950 4400 7950 3950
+	7950 4200 7950 3950
 Connection ~ 7950 3950
 Wire Wire Line
-	8950 4650 8950 4800
-Wire Wire Line
-	8550 4800 8550 4950
-Wire Wire Line
-	8550 4950 9100 4950
-Wire Wire Line
-	8550 4400 8550 3950
+	8550 4200 8550 3950
 Connection ~ 8550 3950
-Connection ~ 9100 4950
 Wire Wire Line
 	7900 1350 7900 6300
@@
 Connection ~ 6750 5150
 Connection ~ 7250 5700
+$Comp
+L DIODE D32
+U 1 1 5740CB82
+P 8150 4600
+F 0 "D32" H 8150 4500 40  0000 C CNN
+F 1 "DIODE" H 8150 4500 40  0001 C CNN
+F 2 "Diodes_SMD:SOD-123" H 8150 4600 60  0001 C CNN
+F 3 "" H 8150 4600 60  0000 C CNN
+	1    8150 4600
+	1    0    0    -1
+$EndComp
+$Comp
+L MX1A S321
+U 1 1 586CD089
+P 8150 4600
+F 0 "S321" H 8000 4850 60  0000 C CNN
+F 1 "MX1A" H 8150 4700 60  0000 C CNN
+F 2 "mx1a:MX1A" H 8150 4600 60  0001 C CNN
+F 3 "" H 8150 4600 60  0000 C CNN
+	1    8150 4600
+	1    0    0    -1
+$EndComp
+Wire Wire Line
+	7950 4600 7950 4750
+Wire Wire Line
+	7950 4750 8500 4750
+Connection ~ 8500 4750
+Wire Wire Line
+	8350 4450 8450 4450
+Connection ~ 8450 4450
+Wire Wire Line
+	8450 4600 8350 4600
+$Comp
+L MX1A S331
+U 1 1 586CDBF9
+P 8750 4600
+F 0 "S331" H 8600 4850 60  0000 C CNN
+F 1 "MX1A" H 8750 4700 60  0000 C CNN
+F 2 "mx1a:MX1A" H 8750 4600 60  0001 C CNN
+F 3 "" H 8750 4600 60  0000 C CNN
+	1    8750 4600
+	1    0    0    -1
+$EndComp
+Wire Wire Line
+	8950 4450 9050 4450
+Connection ~ 9050 4450
+Wire Wire Line
+	8550 4600 8550 4750
+Wire Wire Line
+	8550 4750 9100 4750
+Connection ~ 9100 4750
+Wire Wire Line
+	9050 4600 8950 4600
+Wire Wire Line
+	5850 5650 5950 5650
+Connection ~ 5950 5650
+Wire Wire Line
+	5450 5850 5450 6000
+Wire Wire Line
+	5450 6000 6000 6000
+Connection ~ 6000 6000
+Wire Wire Line
+	5950 5850 5850 5850
+$Comp
+L MX1A S361
+U 1 1 586E55CC
+P 3750 5800
+F 0 "S361" H 3600 6050 60  0000 C CNN
+F 1 "MX1A" H 3750 5900 60  0000 C CNN
+F 2 "mx1a:MX1A" H 3750 5800 60  0001 C CNN
+F 3 "" H 3750 5800 60  0000 C CNN
+	1    3750 5800
+	1    0    0    -1
+$EndComp
+Wire Wire Line
+	3950 5650 4050 5650
+Connection ~ 4050 5650
+Wire Wire Line
+	3550 5400 3550 5150
+Connection ~ 3550 5150
+Wire Wire Line
+	4050 5850 3950 5850
+$Comp
+L MX1A S401
+U 1 1 586E82C5
+P 7500 5800
+F 0 "S401" H 7350 6050 60  0000 C CNN
+F 1 "MX1A" H 7500 5900 60  0000 C CNN
+F 2 "mx1a:MX1A" H 7500 5800 60  0001 C CNN
+F 3 "" H 7500 5800 60  0000 C CNN
+	1    7500 5800
+	1    0    0    -1
+$EndComp
+Wire Wire Line
+	7300 5400 7300 5150
+Connection ~ 7300 5150
+Wire Wire Line
+	7700 5650 7800 5650
+Connection ~ 7800 5650
+Wire Wire Line
+	7800 5850 7700 5850
 $EndSCHEMATC

Commit message: rebuild daisy
Parts:
- D1, D10, D11, D12, D13, D14, D15, D16, D17, D18, D19, D2, D20, D21, D22, D23, D24, D25, D26, D27, D28, D29, D3, D30, D31, D32, D33, D34, D35, D36, D37, D38, D39, D4, D40, D41, D42, D5, D6, D7, D8, D9: footprint Diodes_SMD:SOD-123 -> Diodes_SMD:D_SOD-123
- S1, S10, S11, S12, S13, S14, S15, S16, S17, S18, S19, S2, S20, S21, S22, S23, S24, S25, S26, S27, S28, S29, S3, S30, S31, S32, S321, S33, S331, S34, S35, S36, S361, S37, S38, S381, S39, S4, S40, S401, S41, S42, S5, S6, S7, S8, S9: footprint mx1a:MX1A -> keebs:Mx_Alps_125
