File: keyboard.kicad_pcb (KiCad board)
At the start: 2 copper layers, 229.9 x 77.5 mm, 231 parts, among them IC1 ATMEGA32U4, J1 USBMINI_B05, P1 ISP, P2 GPIO Port, Q1 MOS_P, X1 CRYSTAL

Commit message: 重新画线
Routing:
- net /Row3: track 298.5 -> 0.00 mm, vias 7 -> 0
- net /Row0: track 250.1 -> 0.00 mm, vias 2 -> 0
- net /Row1: track 238.9 -> 0.00 mm, vias 3 -> 0
- net /Row2: track 221.3 -> 0.00 mm, vias 2 -> 0
- net Net-(IC1-Pad4): track 196.0 -> 0.00 mm, vias 6 -> 0
- net Net-(IC1-Pad3): track 177.3 -> 0.00 mm, vias 4 -> 0
- net /GPIO3: track 94.3 -> 0.00 mm, vias 2 -> 0
- net /GPIO2: track 92.9 -> 0.00 mm, vias 2 -> 0
- net /GPIO0: track 89.5 -> 0.00 mm, vias 2 -> 0
- net /GPIO1: track 87.7 -> 0.00 mm, vias 2 -> 0
- net GND: track 80.1 -> 0.00 mm, vias 3 -> 0
- net /Col0: track 65.3 -> 0.00 mm, vias 4 -> 0
- net VCC: track 59.2 -> 0.00 mm, vias 4 -> 0
- net Net-(C2-Pad1): track 40.8 -> 0.00 mm, vias 3 -> 0
- net Net-(C1-Pad1): track 30.7 -> 0.00 mm, vias 3 -> 0
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Other:
- net class Default: via_dia 0.3 -> 0.4; via_drill 0.25 -> 0.2

Commit message: some line
Parts:
- moved D39 2.49 mm to (205.9, 106.4)
Routing:
- net /Row3: track 0.00 -> 303.8 mm, vias 0 -> 2
- net /Row0: track 0.00 -> 250.9 mm, vias 0 -> 4
- net /Row1: track 0.00 -> 240.8 mm, vias 0 -> 4
- net /Row2: track 0.00 -> 227.8 mm, vias 0 -> 2
- net GND: track 0.00 -> 120.5 mm, vias 0 -> 4
- net /GPIO3: track 0.00 -> 96.0 mm, vias 0 -> 2
- net VCC: track 0.00 -> 93.6 mm, vias 0 -> 8
- net /GPIO2: track 0.00 -> 90.3 mm, vias 0 -> 2
- net /GPIO0: track 0.00 -> 88.1 mm, vias 0 -> 2
- net /GPIO1: track 0.00 -> 87.0 mm, vias 0 -> 2
- net /~Res: track 0.00 -> 67.1 mm, vias 0 -> 4
- net Net-(C1-Pad1): track 0.00 -> 36.0 mm, vias 0 -> 3
- net Net-(C2-Pad1): track 0.00 -> 27.3 mm, vias 0 -> 2
- net Net-(J1-Pad2): track 0.00 -> 19.1 mm, vias 0 -> 2
- net Net-(C3-Pad1): track 0.00 -> 16.7 mm, vias 0 -> 2
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Other:
- net class Default: via_dia 0.4 -> 0.6

Commit message: sync
Routing:
- net /ESC: track 0.00 -> 226.0 mm, vias 0 -> 2
- net Net-(IC1-Pad4): track 0.00 -> 190.6 mm, vias 0 -> 3
- net Net-(IC1-Pad3): track 0.00 -> 175.9 mm, vias 0 -> 4
- net VCC: track 93.6 -> 95.5 mm, vias 8 -> 9
- net Net-(C1-Pad1): track 36.0 -> 35.1 mm

Commit message: sync
Routing:
- net /Col6: track 0.00 -> 149.5 mm, vias 0 -> 9
- net /GPIO0: track 88.1 -> 176.9 mm, vias 2 -> 3
- net /GPIO1: track 87.0 -> 157.1 mm, vias 2 -> 5
- net GND: track 120.5 -> 132.7 mm, vias 4 -> 6
- net VCC: track 95.5 -> 106.1 mm, vias 9 -> 11
- net Net-(IC1-Pad33): track 0.00 -> 4.32 mm, vias 1 -> 2
- net Net-(IC1-Pad3): track 175.9 -> 175.0 mm
- net Net-(IC1-Pad4): track 190.6 -> 191.3 mm, vias 3 -> 4

Commit message: rebuild daisy
Parts:
- removed MXLED (x5): HOLE, holes:Mechanical_Hole
- removed MXST (x4): VAL**, mx1a:MXST
- C1, C10, C11, C12, C13, C14, C15, C16, C17, C18, C19, C2, C20, C3, C4, C5, C6, C7, C8, C9, J1, LR1, LR10, LR11, LR12, LR13, LR14, LR15, LR16, LR17, LR18, LR19, LR2, LR20, LR21, LR22, LR23, LR24, LR25, LR26, LR27, LR28, LR29, LR3, LR30, LR31, LR32, LR33, LR34, LR35, LR36, LR37, LR38, LR39, LR4, LR40, LR41, LR42, LR43, LR5, LR6, LR7, LR8, LR9, Q1, R1, R2, R3, R4, R5, RGBLED1, RGBLED10, RGBLED11, RGBLED12, RGBLED2, RGBLED3, RGBLED4, RGBLED5, RGBLED6, RGBLED7, RGBLED8, RGBLED9, X1: moved to F.Cu
- D1, D10, D11, D12, D13, D14, D15, D16, D17, D18, D19, D2, D20, D21, D22, D23, D24, D25, D26, D27, D28, D29, D3, D30, D31, D32, D33, D34, D35, D36, D37, D38, D39, D4, D40, D41, D42, D5, D6, D7, D8, D9: footprint Diodes_SMD:SOD-123 -> Diodes_SMD:D_SOD-123; moved to F.Cu
- IC1: footprint TQFP44:TQFP44 -> Housings_QFP:TQFP-44_10x10mm_Pitch0.8mm; moved to F.Cu
- LED1, LED10, LED11, LED12, LED13, LED14, LED15, LED16, LED17, LED18, LED19, LED2, LED20, LED21, LED22, LED23, LED24, LED25, LED26, LED27, LED28, LED29, LED3, LED30, LED31, LED32, LED33, LED34, LED35, LED36, LED37, LED38, LED39, LED391, LED4, LED40, LED41, LED42, LED5, LED6, LED7, LED8, LED9: footprint mx1a-led:MX1A-led -> mx1a:MX1A-led
- LED331, LED341, LED371, LED411: footprint mx1a-led:MX1A-led -> mx1a:MX1A-led; moved to F.Cu
- P1: footprint Socket_Strips:Socket_Strip_Straight_2x03 -> Socket_Strips:Socket_Strip_Straight_2x03_Pitch2.54mm
- P2: footprint Socket_Strips:Socket_Strip_Straight_1x04 -> Socket_Strips:Socket_Strip_Straight_1x05_Pitch2.54mm
- S1, S10, S11, S12, S13, S14, S15, S16, S17, S18, S19, S2, S20, S21, S22, S23, S24, S25, S26, S27, S28, S29, S3, S30, S31, S32, S321, S33, S331, S34, S35, S36, S361, S39, S4, S40, S401, S41, S42, S5, S6, S7, S8, S9: footprint mx1a:MX1A -> keebs:Mx_Alps_100
- S37: footprint mx1a:MX1A -> keebs:Mx_Alps_225
- S38: footprint 6.25:CHERRY_PCB_625H_Rev -> keebs:Mx_Alps_625
- S381: footprint mx1a:MX1A -> keebs:Mx_Alps_275
- moved LR10 135.0 mm to (144.3, 116.3), turned to 0 degrees
- moved LR12 123.7 mm to (144.3, 116.3), turned to 0 degrees
- moved RGBLED6 122.1 mm to (144.3, 116.3), turned to 0 degrees
- moved LR23 120.1 mm to (144.3, 116.3), turned to 0 degrees
- moved D42 119.5 mm to (144.3, 116.3), turned to 0 degrees
- moved D1 119.2 mm to (144.3, 116.3), turned to 0 degrees
- moved LR9 119.1 mm to (144.3, 116.3), turned to 0 degrees
- moved C14 117.4 mm to (144.3, 116.3), turned to 0 degrees
- moved LR42 115.3 mm to (144.3, 116.3), turned to 0 degrees
- moved J1 115.2 mm to (144.3, 116.3), turned to 0 degrees
- moved LR34 112.4 mm to (144.3, 116.3), turned to 0 degrees
- moved D11 110.8 mm to (144.3, 116.3), turned to 0 degrees
- moved D12 110.7 mm to (144.3, 116.3), turned to 0 degrees
- moved D22 110.2 mm to (144.3, 116.3), turned to 0 degrees
- moved D2 106.8 mm to (144.3, 116.3), turned to 0 degrees
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Connections:
- LED31 pad 1: Net-(LED30-Pad1) -> Net-(LED31-Pad1)
Routing:
- net /Row3: track 303.8 -> 0.00 mm, vias 2 -> 0
- net /Row0: track 250.9 -> 0.00 mm, vias 4 -> 0
- net /Row1: track 240.8 -> 0.00 mm, vias 4 -> 0
- net /Row2: track 227.8 -> 0.00 mm, vias 2 -> 0
- net /ESC: track 226.0 -> 0.00 mm, vias 2 -> 0
- net Net-(IC1-Pad4): track 191.3 -> 0.00 mm, vias 4 -> 0
- net /GPIO0: track 176.9 -> 0.00 mm, vias 3 -> 0
- net Net-(IC1-Pad3): track 175.0 -> 0.00 mm, vias 4 -> 0
- net /GPIO1: track 157.1 -> 0.00 mm, vias 5 -> 0
- net /Col6: track 149.5 -> 0.00 mm, vias 9 -> 0
- net GND: track 132.7 -> 0.00 mm, vias 6 -> 0
- net VCC: track 106.1 -> 0.00 mm, vias 11 -> 0
- net /GPIO3: track 96.0 -> 0.00 mm, vias 2 -> 0
- net /GPIO2: track 90.3 -> 0.00 mm, vias 2 -> 0
- net /~Res: track 67.1 -> 0.00 mm, vias 4 -> 0
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Other:
- board size 229.9 x 77.5 mm -> 228.6 x 76.2 mm
- board text removed: "GND"
- board text removed: "MISO"
- board text removed: "MOSI"
- board text removed: "PB0"
- board text removed: "PB1"
- board text removed: "PB2"
- board text removed: "PD1"
- board text removed: "RES"
- board text removed: "Rev 1.0 Pro"
- board text removed: "SCK"
- board text removed: "USB"
- board text removed: "VCC"

Commit message: 原件摆放完毕
Parts:
- C1, C10, C11, C12, C13, C14, C15, C16, C17, C18, C19, C2, C20, C3, C4, C5, C6, C7, C8, C9, IC1, J1, LR1, LR10, LR11, LR12, LR13, LR14, LR15, LR16, LR17, LR18, LR19, LR2, LR20, LR21, LR22, LR23, LR24, LR25, LR26, LR27, LR28, LR29, LR3, LR30, LR31, LR32, LR33, LR34, LR35, LR36, LR37, LR38, LR39, LR4, LR40, LR41, LR42, LR43, LR5, LR6, LR7, LR8, LR9, Q1, R1, R2, R3, R4, R5, RGBLED1, RGBLED10, RGBLED11, RGBLED12, RGBLED2, RGBLED3, RGBLED4, RGBLED5, RGBLED6, RGBLED7, RGBLED8, RGBLED9: moved to B.Cu
- D1, D10, D11, D12, D13, D14, D15, D16, D17, D18, D19, D2, D20, D21, D22, D23, D24, D25, D26, D27, D28, D29, D3, D30, D31, D32, D33, D34, D35, D36, D37, D38, D39, D4, D40, D41, D42, D5, D6, D7, D8, D9: footprint Diodes_SMD:D_SOD-123 -> Diodes_SMD:D_0805; moved to B.Cu
- X1: footprint Crystals:Crystal_HC49-U_Vertical -> Crystals:Crystal_SMD_5032-2pin_5.0x3.2mm; moved to B.Cu
- moved D1 138.6 mm to (32.8, 34.0), turned to 270 degrees
- moved LR10 134.6 mm to (252.2, 35.8), turned to 90 degrees
- moved LR12 129.6 mm to (42.7, 35.8), turned to 90 degrees
- moved C14 128.6 mm to (253.5, 48.3), turned to 90 degrees
- moved D42 127.9 mm to (242.3, 34.0), turned to 270 degrees
- moved D12 126.0 mm to (35.3, 53.1), turned to 270 degrees
- moved D2 123.7 mm to (51.8, 34.0), turned to 270 degrees
- moved RGBLED6 122.6 mm to (246.6, 48.8), turned to 180 degrees
- moved LR9 119.9 mm to (233.2, 35.8), turned to 90 degrees
- moved LR23 118.0 mm to (245.1, 54.9), turned to 90 degrees
- moved LR11 116.8 mm to (45.0, 54.9), turned to 90 degrees
- moved LR34 115.9 mm to (252.2, 73.9), turned to 90 degrees
- moved LR1 115.3 mm to (61.7, 35.8), turned to 90 degrees
- moved D11 114.0 mm to (223.3, 34.0), turned to 270 degrees
- moved D23 113.4 mm to (39.9, 72.1), turned to 270 degrees
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
Commit message: complete
Parts:
- added REF**: MountingHole_2.2mm_M2_ISO14580_Pad, Mounting_Holes:MountingHole_2.2mm_M2_ISO14580_Pad, F.Cu at (49.0, 87.2)
- added REF**: MountingHole_2.2mm_M2_ISO14580_Pad, Mounting_Holes:MountingHole_2.2mm_M2_ISO14580_Pad, F.Cu at (144.3, 87.2)
- added REF**: MountingHole_2.2mm_M2_ISO14580_Pad, Mounting_Holes:MountingHole_2.2mm_M2_ISO14580_Pad, F.Cu at (239.6, 87.2)
- added REF**: MountingHole_2.2mm_M2_ISO14580_Pad, Mounting_Holes:MountingHole_2.2mm_M2_ISO14580_Pad, F.Cu at (239.6, 49.0)
- added REF**: MountingHole_2.2mm_M2_ISO14580_Pad, Mounting_Holes:MountingHole_2.2mm_M2_ISO14580_Pad, F.Cu at (144.3, 49.0)
- added REF**: MountingHole_2.2mm_M2_ISO14580_Pad, Mounting_Holes:MountingHole_2.2mm_M2_ISO14580_Pad, F.Cu at (49.0, 49.0)
- moved R2 2.79 mm to (143.3, 43.9)
- moved R1 2.54 mm to (145.3, 43.9)
- moved C17 2.54 mm to (177.5, 82.0)
- moved R5 2.34 mm to (189.2, 87.9), turned to 0 degrees
- moved X1 1.30 mm to (193.5, 95.5)
- moved C1 1.27 mm to (193.3, 91.2)
- moved C2 1.27 mm to (193.3, 100.3)
- moved R3 1.27 mm to (193.3, 103.6)
- moved IC1 0.80 mm to (184.4, 96.5)
- moved C3 0.25 mm to (184.7, 86.9)
- turned RGBLED10 to 0 degrees
- turned RGBLED11 to 0 degrees
- turned RGBLED12 to 0 degrees
- turned RGBLED7 to 0 degrees
- turned RGBLED8 to 0 degrees
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Routing:
- net GND: track 0.00 -> 1189.0 mm, vias 0 -> 41
- net /led/LRow0: track 0.00 -> 833.9 mm, vias 0 -> 11
- net VCC: track 0.00 -> 765.3 mm, vias 0 -> 25
- net /Row3: track 0.00 -> 289.1 mm, vias 0 -> 1
- net /Row0: track 0.00 -> 276.7 mm, vias 0 -> 4
- net /Row1: track 0.00 -> 271.6 mm, vias 0 -> 2
- net /Row2: track 0.00 -> 268.8 mm, vias 0 -> 3
- net /Col0: track 0.00 -> 229.5 mm, vias 0 -> 6
- net /WASD: track 0.00 -> 216.3 mm, vias 0 -> 5
- net /Col1: track 0.00 -> 214.4 mm, vias 0 -> 12
- net /ESC: track 0.00 -> 206.9 mm, vias 0 -> 6
- net /Col3: track 0.00 -> 190.7 mm, vias 0 -> 11
- net /Col10: track 0.00 -> 189.4 mm, vias 0 -> 6
- net /Col2: track 0.00 -> 188.6 mm, vias 0 -> 11
- net /Caps: track 0.00 -> 182.6 mm, vias 0 -> 5
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Other:
- outline, holes or cut-outs redrawn
- net class Default: via_drill 0.2 -> 0.4
- rule trace_min: 0.2 -> 0.25
- rule via_min_size: 0.1 -> 0.6
