File: led.sch (KiCad schematic (older format))
At the start: 117 parts, among them Q1 MOS_P

Commit message: Final touches on schematic & Clean up PCB
Parts:
- renumbered LR41 to LR43
Changed lines of the file:
@@
 $EndComp
 $Comp
-L R LR41
+L R LR43
 U 1 1 5741986A
 P 2550 8650
-F 0 "LR41" V 2630 8650 50  0000 C CNN
+F 0 "LR43" V 2630 8650 50  0000 C CNN
 F 1 "330R" V 2550 8650 50  0000 C CNN
 F 2 "Resistors_SMD:R_0805" H 2550 8650 60  0001 C CNN

Commit message: Layout
Parts:
- removed LR331, LR341, LR391: 330R, Resistors_SMD:R_0805, symbol R
- added LED371, LED411: LED, mx1a:MX1A-led, symbol LED
Connections:
- wire segments 305 -> 303
Other:
- moved on the sheet: LED331, LED341, LED391
Changed lines of the file:
@@
 $EndComp
 $Comp
-L VCC #PWR022
+L VCC #PWR021
 U 1 1 574CA66F
 P 3950 9100
-F 0 "#PWR022" H 3950 9200 30  0001 C CNN
+F 0 "#PWR021" H 3950 9200 30  0001 C CNN
 F 1 "VCC" H 3950 9200 30  0000 C CNN
 F 2 "" H 3950 9100 60  0000 C CNN
@@
 $EndComp
 $Comp
-L GND #PWR023
+L GND #PWR022
 U 1 1 576B3C00
 P 4550 1950
-F 0 "#PWR023" H 4550 1950 30  0001 C CNN
+F 0 "#PWR022" H 4550 1950 30  0001 C CNN
 F 1 "GND" H 4550 1880 30  0001 C CNN
 F 2 "" H 4550 1950 60  0000 C CNN
@@
 $EndComp
 $Comp
-L GND #PWR024
+L GND #PWR023
 U 1 1 576B6379
 P 5350 1950
-F 0 "#PWR024" H 5350 1950 30  0001 C CNN
+F 0 "#PWR023" H 5350 1950 30  0001 C CNN
 F 1 "GND" H 5350 1880 30  0001 C CNN
 F 2 "" H 5350 1950 60  0000 C CNN
@@
 $EndComp
 $Comp
-L GND #PWR025
+L GND #PWR024
 U 1 1 576B64B9
 P 6150 1950
-F 0 "#PWR025" H 6150 1950 30  0001 C CNN
+F 0 "#PWR024" H 6150 1950 30  0001 C CNN
 F 1 "GND" H 6150 1880 30  0001 C CNN
 F 2 "" H 6150 1950 60  0000 C CNN
@@
 $EndComp
 $Comp
-L GND #PWR026
+L GND #PWR025
 U 1 1 576B9647
 P 6950 1950
-F 0 "#PWR026" H 6950 1950 30  0001 C CNN
+F 0 "#PWR025" H 6950 1950 30  0001 C CNN
 F 1 "GND" H 6950 1880 30  0001 C CNN
 F 2 "" H 6950 1950 60  0000 C CNN
@@
 $EndComp
 $Comp
-L GND #PWR027
+L GND #PWR026
 U 1 1 576B9787
 P 7750 1950
-F 0 "#PWR027" H 7750 1950 30  0001 C CNN
+F 0 "#PWR026" H 7750 1950 30  0001 C CNN
 F 1 "GND" H 7750 1880 30  0001 C CNN
 F 2 "" H 7750 1950 60  0000 C CNN
@@
 $EndComp
 $Comp
-L GND #PWR028
+L GND #PWR027
 U 1 1 576BA13A
 P 8550 1950
-F 0 "#PWR028" H 8550 1950 30  0001 C CNN
+F 0 "#PWR027" H 8550 1950 30  0001 C CNN
 F 1 "GND" H 8550 1880 30  0001 C CNN
 F 2 "" H 8550 1950 60  0000 C CNN
@@
 $EndComp
 $Comp
-L GND #PWR029
+L GND #PWR028
 U 1 1 576BA27A
 P 9350 1950
-F 0 "#PWR029" H 9350 1950 30  0001 C CNN
+F 0 "#PWR028" H 9350 1950 30  0001 C CNN
 F 1 "GND" H 9350 1880 30  0001 C CNN
 F 2 "" H 9350 1950 60  0000 C CNN
@@
 $EndComp
 $Comp
-L GND #PWR030
+L GND #PWR029
 U 1 1 576BA3BA
 P 10150 1950
-F 0 "#PWR030" H 10150 1950 30  0001 C CNN
+F 0 "#PWR029" H 10150 1950 30  0001 C CNN
 F 1 "GND" H 10150 1880 30  0001 C CNN
 F 2 "" H 10150 1950 60  0000 C CNN
@@
 $EndComp
 $Comp
-L GND #PWR031
+L GND #PWR030
 U 1 1 576BB1DA
 P 10950 1950
-F 0 "#PWR031" H 10950 1950 30  0001 C CNN
+F 0 "#PWR030" H 10950 1950 30  0001 C CNN
 F 1 "GND" H 10950 1880 30  0001 C CNN
 F 2 "" H 10950 1950 60  0000 C CNN
@@
 $EndComp
 $Comp
-L GND #PWR032
+L GND #PWR031
 U 1 1 576BB31A
 P 11750 1950
-F 0 "#PWR032" H 11750 1950 30  0001 C CNN
+F 0 "#PWR031" H 11750 1950 30  0001 C CNN
 F 1 "GND" H 11750 1880 30  0001 C CNN
 F 2 "" H 11750 1950 60  0000 C CNN
@@
 $EndComp
 $Comp
-L GND #PWR033
+L GND #PWR032
 U 1 1 576BB45A
 P 12550 1950
-F 0 "#PWR033" H 12550 1950 30  0001 C CNN
+F 0 "#PWR032" H 12550 1950 30  0001 C CNN
 F 1 "GND" H 12550 1880 30  0001 C CNN
 F 2 "" H 12550 1950 60  0000 C CNN
@@
 $EndComp
 $Comp
-L GND #PWR034
+L GND #PWR033
 U 1 1 576BB59A
 P 13400 1950
-F 0 "#PWR034" H 13400 1950 30  0001 C CNN
+F 0 "#PWR033" H 13400 1950 30  0001 C CNN
 F 1 "GND" H 13400 1880 30  0001 C CNN
 F 2 "" H 13400 1950 60  0000 C CNN
@@
 $EndComp
 $Comp
-L VCC #PWR035
+L VCC #PWR034
 U 1 1 57711906
 P 2600 4850
-F 0 "#PWR035" H 2600 4950 30  0001 C CNN
+F 0 "#PWR034" H 2600 4950 30  0001 C CNN
 F 1 "VCC" H 2600 4950 30  0000 C CNN
 F 2 "" H 2600 4850 60  0000 C CNN
@@
 NoConn ~ 16000 8400
 $Comp
-L GND #PWR036
+L GND #PWR035
 U 1 1 576B1DB9
 P 16650 7850
-F 0 "#PWR036" H 16650 7850 30  0001 C CNN
+F 0 "#PWR035" H 16650 7850 30  0001 C CNN
 F 1 "GND" H 16650 7780 30  0001 C CNN
 F 2 "" H 16650 7850 60  0000 C CNN
@@
 $EndComp
 $Comp
-L VCC #PWR037
+L VCC #PWR036
 U 1 1 57794F60
 P 15750 2200
-F 0 "#PWR037" H 15750 2300 30  0001 C CNN
+F 0 "#PWR036" H 15750 2300 30  0001 C CNN
 F 1 "VCC" H 15750 2300 30  0000 C CNN
 F 2 "" H 15750 2200 60  0000 C CNN
@@
 $EndComp
 $Comp
-L VCC #PWR038
+L VCC #PWR037
 U 1 1 5779508F
 P 16450 2200
-F 0 "#PWR038" H 16450 2300 30  0001 C CNN
+F 0 "#PWR037" H 16450 2300 30  0001 C CNN
 F 1 "VCC" H 16450 2300 30  0000 C CNN
 F 2 "" H 16450 2200 60  0000 C CNN
@@
 $EndComp
 $Comp
-L VCC #PWR039
+L VCC #PWR038
 U 1 1 577951B7
 P 17650 2200
-F 0 "#PWR039" H 17650 2300 30  0001 C CNN
+F 0 "#PWR038" H 17650 2300 30  0001 C CNN
 F 1 "VCC" H 17650 2300 30  0000 C CNN
 F 2 "" H 17650 2200 60  0000 C CNN
@@
 $EndComp
 $Comp
-L R LR391
-U 1 1 586D5739
-P 9250 6150
-F 0 "LR391" V 9330 6150 50  0000 C CNN
-F 1 "330R" V 9250 6150 50  0000 C CNN
-F 2 "Resistors_SMD:R_0805" H 9250 6150 60  0001 C CNN
-F 3 "" H 9250 6150 60  0000 C CNN
-	1    9250 6150
-	1    0    0    -1
-$EndComp
-$Comp
 L LED LED391
 U 1 1 586D5743
-P 8950 6450
-F 0 "LED391" H 8950 6550 50  0000 C CNN
-F 1 "LED" H 8950 6350 50  0000 C CNN
-F 2 "mx1a:MX1A-led" H 8950 6450 60  0001 C CNN
-F 3 "" H 8950 6450 60  0000 C CNN
-	1    8950 6450
+P 8900 6150
+F 0 "LED391" H 8900 6250 50  0000 C CNN
+F 1 "LED" H 8900 6050 50  0000 C CNN
+F 2 "mx1a:MX1A-led" H 8900 6150 60  0001 C CNN
+F 3 "" H 8900 6150 60  0000 C CNN
+	1    8900 6150
 	-1   0    0    1
 $EndComp
@@
 	12300 4500 12400 4500
 Wire Wire Line
-	12400 4500 12400 4450
+	12400 4450 12400 4800
 Wire Wire Line
 	12400 3850 12400 3950
@@
 	13100 4500 13200 4500
 Wire Wire Line
-	13200 4500 13200 4450
+	13200 4450 13200 4800
 Wire Wire Line
 	13200 3850 13200 3950
@@
 	6700 5850 6800 5850
 Wire Wire Line
-	6800 5850 6800 5800
+	6800 5800 6800 6150
 Wire Wire Line
 	6800 5200 6800 5300
@@
 	11500 5850 11600 5850
 Wire Wire Line
-	11600 5850 11600 5800
+	11600 5800 11600 6150
 Wire Wire Line
 	11600 5200 11600 5300
@@
 	9200 5200 9200 5300
 Wire Wire Line
-	9200 5850 9200 5800
+	9200 5800 9200 6150
 Wire Wire Line
 	9100 5850 9200 5850
@@
 	8300 5850 8400 5850
 Connection ~ 8400 5200
-Wire Wire Line
-	8550 6450 8750 6450
-Wire Wire Line
-	9250 5200 9250 5900
-Wire Wire Line
-	9250 6450 9250 6400
-Wire Wire Line
-	9150 6450 9250 6450
-Connection ~ 9250 5200
-Connection ~ 8550 6450
 Connection ~ 7750 5850
-$Comp
-L R LR331
-U 1 1 586DDF79
-P 12500 4750
-F 0 "LR331" V 12580 4750 50  0000 C CNN
-F 1 "330R" V 12500 4750 50  0000 C CNN
-F 2 "Resistors_SMD:R_0805" H 12500 4750 60  0001 C CNN
-F 3 "" H 12500 4750 60  0000 C CNN
-	1    12500 4750
-	1    0    0    -1
-$EndComp
 $Comp
 L LED LED331
 U 1 1 586DDF7F
-P 12200 5050
-F 0 "LED331" H 12200 5150 50  0000 C CNN
-F 1 "LED" H 12200 4950 50  0000 C CNN
-F 2 "mx1a:MX1A-led" H 12200 5050 60  0001 C CNN
-F 3 "" H 12200 5050 60  0000 C CNN
-	1    12200 5050
-	-1   0    0    1
-$EndComp
-Wire Wire Line
-	12400 5050 12500 5050
-Wire Wire Line
-	12500 5050 12500 5000
-Wire Wire Line
-	12500 3850 12500 4500
-Wire Wire Line
-	11750 5050 12000 5050
-Connection ~ 12500 3850
-Connection ~ 11750 5050
-$Comp
-L R LR341
-U 1 1 586DE4F5
-P 13350 4750
-F 0 "LR341" V 13430 4750 50  0000 C CNN
-F 1 "330R" V 13350 4750 50  0000 C CNN
-F 2 "Resistors_SMD:R_0805" H 13350 4750 60  0001 C CNN
-F 3 "" H 13350 4750 60  0000 C CNN
-	1    13350 4750
-	1    0    0    -1
+P 12100 4800
+F 0 "LED331" H 12100 4900 50  0000 C CNN
+F 1 "LED" H 12100 4700 50  0000 C CNN
+F 2 "mx1a:MX1A-led" H 12100 4800 60  0001 C CNN
+F 3 "" H 12100 4800 60  0000 C CNN
+	1    12100 4800
+	-1   0    0    1
 $EndComp
 $Comp
 L LED LED341
 U 1 1 586DE4FB
-P 13050 5050
-F 0 "LED341" H 13050 5150 50  0000 C CNN
-F 1 "LED" H 13050 4950 50  0000 C CNN
-F 2 "mx1a:MX1A-led" H 13050 5050 60  0001 C CNN
-F 3 "" H 13050 5050 60  0000 C CNN
-	1    13050 5050
-	-1   0    0    1
-$EndComp
-Wire Wire Line
-	13250 5050 13350 5050
-Wire Wire Line
-	13350 5050 13350 5000
-Wire Wire Line
-	13350 3850 13350 4500
-Wire Wire Line
-	12550 5050 12850 5050
-Connection ~ 12550 5050
+P 12900 4800
+F 0 "LED341" H 12900 4900 50  0000 C CNN
+F 1 "LED" H 12900 4700 50  0000 C CNN
+F 2 "mx1a:MX1A-led" H 12900 4800 60  0001 C CNN
+F 3 "" H 12900 4800 60  0000 C CNN
+	1    12900 4800
+	-1   0    0    1
+$EndComp
 Connection ~ 13350 3850
 Wire Wire Line
 	7750 5850 7900 5850
+Wire Wire Line
+	12700 4800 12550 4800
+Connection ~ 12550 4800
+Wire Wire Line
+	13200 4800 13100 4800
+Connection ~ 13200 4500
+Wire Wire Line
+	8700 6150 8550 6150
+Connection ~ 8550 6150
+Wire Wire Line
+	9200 6150 9100 6150
+Connection ~ 9200 5850
+Wire Wire Line
+	11750 4800 11900 4800
+Connection ~ 11750 4800
+Wire Wire Line
+	12400 4800 12300 4800
+Connection ~ 12400 4500
+$Comp
+L LED LED371
+U 1 1 586E6C65
+P 6500 6150
+F 0 "LED371" H 6500 6250 50  0000 C CNN
+F 1 "LED" H 6500 6050 50  0000 C CNN
+F 2 "mx1a:MX1A-led" H 6500 6150 60  0001 C CNN
+F 3 "" H 6500 6150 60  0000 C CNN
+	1    6500 6150
+	-1   0    0    1
+$EndComp
+Wire Wire Line
+	6300 6150 6150 6150
+Connection ~ 6150 6150
+Wire Wire Line
+	6800 6150 6700 6150
+Connection ~ 6800 5850
+$Comp
+L LED LED411
+U 1 1 586E93C6
+P 11300 6150
+F 0 "LED411" H 11300 6250 50  0000 C CNN
+F 1 "LED" H 11300 6050 50  0000 C CNN
+F 2 "mx1a:MX1A-led" H 11300 6150 60  0001 C CNN
+F 3 "" H 11300 6150 60  0000 C CNN
+	1    11300 6150
+	-1   0    0    1
+$EndComp
+Wire Wire Line
+	11100 6150 10950 6150
+Connection ~ 10950 6150
+Wire Wire Line
+	11600 6150 11500 6150
+Connection ~ 11600 5850
 $EndSCHEMATC

Commit message: Redesign v0.3
Parts:
- removed C16, C17, C19, C20: 100nF, Capacitors_SMD:C_0805, symbol Csmall
- removed LED331, LED341, LED371, LED411: LED, mx1a:MX1A-led, symbol LED
- removed LR43: 330R, Resistors_SMD:R_0805, symbol R
- removed RGBLED10, RGBLED11, RGBLED12, RGBLED9: WS2812B, WS2812B:WS2812B, symbol WS2812B
- added JP10, JP11, JP12, JP13, JP14, JP15, JP16, JP17, JP18, JP19, JP5, JP6, JP7, JP8, JP9: JUMPER, passives:Jumper_SMD_2Pads_NC_V, symbol JUMPER
- added JP3, JP4: JUMPER3, passives:Jumper_SMD_3Pads_NC12, symbol JUMPER3
- added LR1, LR12: 330R, resistors:R_0805_V1, symbol R
- C11: renamed from C9; footprint Capacitors_SMD:C_0805 -> capacitors:C_0805
- C12: renamed from C10; footprint Capacitors_SMD:C_0805 -> capacitors:C_0805
- C13: renamed from C11; footprint Capacitors_SMD:C_0805 -> capacitors:C_0805
- C14: renamed from C12; footprint Capacitors_SMD:C_0805 -> capacitors:C_0805
- C15: renamed from C13; footprint Capacitors_SMD:C_0805 -> capacitors:C_0805
- C16: renamed from C14; footprint Capacitors_SMD:C_0805 -> capacitors:C_0805
- C17: renamed from C15; footprint Capacitors_SMD:C_0805 -> capacitors:C_0805
- C18: footprint Capacitors_SMD:C_0805 -> capacitors:C_0805
- LED1: renamed from LED12; footprint mx1a:MX1A-led -> leds:MX1A_LED_Polar
- LED10: renamed from LED8; footprint mx1a:MX1A-led -> leds:MX1A_LED_Polar
- LED11: renamed from LED9; footprint mx1a:MX1A-led -> leds:MX1A_LED_Polar
- LED12: renamed from LED11; footprint mx1a:MX1A-led -> leds:MX1A_LED_Polar
- LED13: renamed from LED14; footprint mx1a:MX1A-led -> leds:MX1A_LED_Polar
- LED14: renamed from LED15; footprint mx1a:MX1A-led -> leds:MX1A_LED_Polar
- LED15: renamed from LED16; footprint mx1a:MX1A-led -> leds:MX1A_LED_Polar
- LED16: renamed from LED17; footprint mx1a:MX1A-led -> leds:MX1A_LED_Polar
- LED17: renamed from LED18; footprint mx1a:MX1A-led -> leds:MX1A_LED_Polar
- LED18: renamed from LED19; footprint mx1a:MX1A-led -> leds:MX1A_LED_Polar
- LED19: renamed from LED20; footprint mx1a:MX1A-led -> leds:MX1A_LED_Polar
- LED2: renamed from LED1; footprint mx1a:MX1A-led -> leds:MX1A_LED_Polar
- LED20: renamed from LED21; footprint mx1a:MX1A-led -> leds:MX1A_LED_Polar
- LED21: renamed from LED22; footprint mx1a:MX1A-led -> leds:MX1A_LED_Polar
- LED22: renamed from LED23; footprint mx1a:MX1A-led -> leds:MX1A_LED_Polar
- LED23: renamed from LED24; footprint mx1a:MX1A-led -> leds:MX1A_LED_Polar
- LED24: renamed from LED25; footprint mx1a:MX1A-led -> leds:MX1A_LED_Polar
- LED25: renamed from LED26; footprint mx1a:MX1A-led -> leds:MX1A_LED_Polar
- LED26: renamed from LED27; footprint mx1a:MX1A-led -> leds:MX1A_LED_Polar
- LED27: renamed from LED28; footprint mx1a:MX1A-led -> leds:MX1A_LED_Polar
- LED28: renamed from LED29; footprint mx1a:MX1A-led -> leds:MX1A_LED_Polar
- LED29: renamed from LED30; footprint mx1a:MX1A-led -> leds:MX1A_LED_Polar
- LED3: renamed from LED13; footprint mx1a:MX1A-led -> leds:MX1A_LED_Polar
- LED30: renamed from LED31; footprint mx1a:MX1A-led -> leds:MX1A_LED_Polar
- LED31: renamed from LED32; footprint mx1a:MX1A-led -> leds:MX1A_LED_Polar
- LED32: renamed from LED33; footprint mx1a:MX1A-led -> leds:MX1A_LED_Polar_Dual
- LED33: renamed from LED34; footprint mx1a:MX1A-led -> leds:MX1A_LED_Polar_Dual
- LED34: renamed from LED35; footprint mx1a:MX1A-led -> leds:MX1A_LED_Polar
- LED35: renamed from LED36; footprint mx1a:MX1A-led -> leds:MX1A_LED_Polar
- LED36: renamed from LED37; footprint mx1a:MX1A-led -> leds:MX1A_LED_Polar_Dual
- LED37: renamed from LED38; footprint mx1a:MX1A-led -> leds:MX1A_LED_Polar
- LED38: renamed from LED39; footprint mx1a:MX1A-led -> leds:MX1A_LED_Polar
- LED38_625: renamed from LED391; footprint mx1a:MX1A-led -> leds:MX1A_LED_Polar
- LED39: renamed from LED40; footprint mx1a:MX1A-led -> leds:MX1A_LED_Polar
- LED4: renamed from LED2; footprint mx1a:MX1A-led -> leds:MX1A_LED_Polar
- LED40: renamed from LED41; footprint mx1a:MX1A-led -> leds:MX1A_LED_Polar_Dual
- LED41: renamed from LED42; footprint mx1a:MX1A-led -> leds:MX1A_LED_Polar
- LED42: renamed from LED10; footprint mx1a:MX1A-led -> leds:MX1A_LED_Polar
- LED5: renamed from LED3; footprint mx1a:MX1A-led -> leds:MX1A_LED_Polar
- LED6: renamed from LED4; footprint mx1a:MX1A-led -> leds:MX1A_LED_Polar
- LED7: renamed from LED5; footprint mx1a:MX1A-led -> leds:MX1A_LED_Polar
- LED8: renamed from LED6; footprint mx1a:MX1A-led -> leds:MX1A_LED_Polar
- LED9: renamed from LED7; footprint mx1a:MX1A-led -> leds:MX1A_LED_Polar
- LR1-2: renamed from LR12; footprint Resistors_SMD:R_0805 -> resistors:R_0805_NA
- LR10: renamed from LR8; footprint Resistors_SMD:R_0805 -> resistors:R_0805_V1
- LR11: renamed from LR9; footprint Resistors_SMD:R_0805 -> resistors:R_0805_V1
- LR12-2: renamed from LR11; footprint Resistors_SMD:R_0805 -> resistors:R_0805_NA
- LR13: renamed from LR14; footprint Resistors_SMD:R_0805 -> resistors:R_0805_V1
- LR14: renamed from LR15; footprint Resistors_SMD:R_0805 -> resistors:R_0805_V1
- LR15: renamed from LR16; footprint Resistors_SMD:R_0805 -> resistors:R_0805_V1
- LR16: renamed from LR17; footprint Resistors_SMD:R_0805 -> resistors:R_0805_V1
- LR17: renamed from LR18; footprint Resistors_SMD:R_0805 -> resistors:R_0805_V1
- LR18: renamed from LR19; footprint Resistors_SMD:R_0805 -> resistors:R_0805_V1
- LR19: renamed from LR20; footprint Resistors_SMD:R_0805 -> resistors:R_0805_V1
- LR2: renamed from LR1; footprint Resistors_SMD:R_0805 -> resistors:R_0805_V1
- LR20: renamed from LR21; footprint Resistors_SMD:R_0805 -> resistors:R_0805_V1
- LR21: renamed from LR22; footprint Resistors_SMD:R_0805 -> resistors:R_0805_V1
- LR22: renamed from LR23; footprint Resistors_SMD:R_0805 -> resistors:R_0805_V1
- LR23: renamed from LR24; footprint Resistors_SMD:R_0805 -> resistors:R_0805_V1
- LR24: renamed from LR25; footprint Resistors_SMD:R_0805 -> resistors:R_0805_V1
- LR25: renamed from LR26; footprint Resistors_SMD:R_0805 -> resistors:R_0805_V1
- LR26: renamed from LR27; footprint Resistors_SMD:R_0805 -> resistors:R_0805_V1
- LR27: renamed from LR28; footprint Resistors_SMD:R_0805 -> resistors:R_0805_V1
- LR28: renamed from LR29; footprint Resistors_SMD:R_0805 -> resistors:R_0805_V1
- LR29: renamed from LR30; footprint Resistors_SMD:R_0805 -> resistors:R_0805_V1
- LR3: renamed from LR13; footprint Resistors_SMD:R_0805 -> resistors:R_0805_V1
- LR30: renamed from LR31; footprint Resistors_SMD:R_0805 -> resistors:R_0805_V1
- LR31: renamed from LR32; footprint Resistors_SMD:R_0805 -> resistors:R_0805_V1
- LR32: renamed from LR33; footprint Resistors_SMD:R_0805 -> resistors:R_0805_V1
- LR33: renamed from LR34; footprint Resistors_SMD:R_0805 -> resistors:R_0805_V1
- LR34: renamed from LR35; footprint Resistors_SMD:R_0805 -> resistors:R_0805_V1
- LR35: renamed from LR36; footprint Resistors_SMD:R_0805 -> resistors:R_0805_V1
- LR36: renamed from LR37; footprint Resistors_SMD:R_0805 -> resistors:R_0805_V1
- LR37: renamed from LR38; footprint Resistors_SMD:R_0805 -> resistors:R_0805_V1
- LR38: renamed from LR39; footprint Resistors_SMD:R_0805 -> resistors:R_0805_V1
- LR39: renamed from LR40; footprint Resistors_SMD:R_0805 -> resistors:R_0805_V1
- LR4: renamed from LR2; footprint Resistors_SMD:R_0805 -> resistors:R_0805_V1
- LR40: renamed from LR41; footprint Resistors_SMD:R_0805 -> resistors:R_0805_V1
- LR41: renamed from LR42; footprint Resistors_SMD:R_0805 -> resistors:R_0805_V1
- LR42: renamed from LR10; footprint Resistors_SMD:R_0805 -> resistors:R_0805_V1
- LR5: renamed from LR3; footprint Resistors_SMD:R_0805 -> resistors:R_0805_V1
- LR6: renamed from LR4; footprint Resistors_SMD:R_0805 -> resistors:R_0805_V1
- LR7: renamed from LR5; footprint Resistors_SMD:R_0805 -> resistors:R_0805_V1
- LR8: renamed from LR6; footprint Resistors_SMD:R_0805 -> resistors:R_0805_V1
- LR9: renamed from LR7; footprint Resistors_SMD:R_0805 -> resistors:R_0805_V1
- Q1: footprint SI2305:SOT-23 -> transistors:SOT-23; symbol MOS_P -> Q_PMOS_GSD
- R4: footprint Resistors_SMD:R_0805 -> resistors:R_0805
- RGBLED1, RGBLED2, RGBLED3, RGBLED4, RGBLED5, RGBLED6, RGBLED7, RGBLED8: footprint WS2812B:WS2812B -> leds:WS2812B
Connections:
- net labels added: Esc, LCol0, LCol1, LCol10, LCol2, LCol3, LCol4, LCol5, LCol6, LCol7, LCol8, LCol9, LVCC, RGB
- net labels removed: Bottom, ESC, WASD
- wire segments 303 -> 300
Other:
- note added: "Dual"
- note added: "Esc"
- note removed: "ESC\n"
- note removed: "WASD"
- moved on the sheet: C11, C12, C13, C14, C15, C16, C17, LED1, LED10, LED11, LED12, LED13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
